Commit message: Align FR3 camera mount and real extrinsics with simulation

File: vendor/fr3_d435i/urdf/fr3_d435i_official.urdf (robot description, URDF)
Before this commit: robot fr3, 33 links, 32 joints
Joints:
- joint d435i_mount_joint: origin xyz=0.0635832488467 0.04912 0.0378225720135 rpy=0 -2.00712863979 0 -> xyz=0.0635832488467 0.01412 0.0378225720135 rpy=3.141592653589793 -2.00712863979 0
